Commit message: hast la vista, socket!

File: install/robomaster_description/share/robomaster_description/urdf/robomaster_ep.urdf.xacro (robot description, xacro)
@@ -17,4 +17,5 @@
   <xacro:include filename="extension.urdf.xacro"/>
   <xacro:include filename="tof.urdf.xacro"/>
+  <xacro:include filename="lidar.urdf.xacro"/>
   <xacro:base tf_prefix="${tf_prefix}"/>
   <xacro:extension tf_prefix="${tf_prefix}" use_rear_extension="true"/>

File: model.urdf (robot description, URDF)
Before this commit: robot robomaster_ep, 43 links, 42 joints
Links:
- added link lidar_link; visual cylinder length=0.05 radius=0.05
Joints:
- added joint lidar_joint: type fixed, parent base_link, child lidar_link, origin xyz=-0.1 0 0.33 rpy=0 0 0
